Commit message: added transformation to body frame for velocity, added endeffector frames in spot.urdf

File: files/spot.urdf (robot description, URDF)
Before this commit: robot spot, 16 links, 15 joints
Links:
- added link front_left_foot, mass 0.0
- added link front_right_foot, mass 0.0
- added link rear_left_foot, mass 0.0
- added link rear_right_foot, mass 0.0
Joints:
- added joint front_left_ankle: type fixed, parent front_left_lower_leg, child front_left_foot, origin xyz=0 0 -0.35 rpy=0 0 0, limit lower=-10 upper=10 effort=1000 velocity=1000
- added joint front_right_ankle: type fixed, parent front_right_lower_leg, child front_right_foot, origin xyz=0 0 -0.35 rpy=0 0 0, limit lower=-10 upper=10 effort=1000 velocity=1000
- added joint rear_left_ankle: type fixed, parent rear_left_lower_leg, child rear_left_foot, origin xyz=0 0 -0.35 rpy=0 0 0, limit lower=-10 upper=10 effort=1000 velocity=1000
- added joint rear_right_ankle: type fixed, parent rear_right_lower_leg, child rear_right_foot, origin xyz=0 0 -0.35 rpy=0 0 0, limit lower=-10 upper=10 effort=1000 velocity=1000
