Commit message: add go1 identification

File: files/go1_description/go1.urdf (robot description, URDF)
Before this commit: robot go1, 46 links, 45 joints
Links:
- removed link camera_chin
- removed link camera_face
- removed link camera_laserscan_link_left
- removed link camera_laserscan_link_right
- removed link camera_left
- removed link camera_optical_chin
- removed link camera_optical_face
- removed link camera_optical_left
- removed link camera_optical_rearDown
- removed link camera_optical_right
- removed link camera_rearDown
- removed link camera_right
- removed link ultraSound_face
- removed link ultraSound_left
- removed link ultraSound_right
- link FL_calf: geometry collision box size=0.213 0.016 0.016; visual mesh filename=/home/khorshidi/mpc_devel/workspace/src/robot_properties_go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 scale=1 1 1
- link FL_hip: geometry collision cylinder length=0.04 radius=0.046; visual mesh filename=/home/khorshidi/mpc_devel/workspace/src/robot_properties_go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 scale=1 1 1
- link FL_thigh: geometry collision box size=0.213 0.0245 0.034; visual mesh filename=/home/khorshidi/mpc_devel/workspace/src/robot_properties_go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 scale=1 1 1
- link FR_calf: geometry collision box size=0.213 0.016 0.016; visual mesh filename=/home/khorshidi/mpc_devel/workspace/src/robot_properties_go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 scale=1 1 1
- link FR_hip: geometry collision cylinder length=0.04 radius=0.046; visual mesh filename=/home/khorshidi/mpc_devel/workspace/src/robot_properties_go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 scale=1 1 1
- link FR_thigh: geometry collision box size=0.213 0.0245 0.034; visual mesh filename=/home/khorshidi/mpc_devel/workspace/src/robot_properties_go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 scale=1 1 1
- link RL_calf: geometry collision box size=0.213 0.016 0.016; visual mesh filename=/home/khorshidi/mpc_devel/workspace/src/robot_properties_go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 scale=1 1 1
- link RL_hip: geometry collision cylinder length=0.04 radius=0.046; visual mesh filename=/home/khorshidi/mpc_devel/workspace/src/robot_properties_go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 scale=1 1 1
- link RL_thigh: geometry collision box size=0.213 0.0245 0.034; visual mesh filename=/home/khorshidi/mpc_devel/workspace/src/robot_properties_go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 scale=1 1 1
- link RR_calf: geometry collision box size=0.213 0.016 0.016; visual mesh filename=/home/khorshidi/mpc_devel/workspace/src/robot_properties_go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 scale=1 1 1
- link RR_hip: geometry collision cylinder length=0.04 radius=0.046; visual mesh filename=/home/khorshidi/mpc_devel/workspace/src/robot_properties_go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 scale=1 1 1
- link RR_thigh: geometry collision box size=0.213 0.0245 0.034; visual mesh filename=/home/khorshidi/mpc_devel/workspace/src/robot_properties_go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 scale=1 1 1
- link trunk: geometry collision box size=0.3762 0.0935 0.114; visual mesh filename=/home/khorshidi/mpc_devel/workspace/src/robot_properties_go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 scale=1 1 1
Joints:
- removed joint camera_joint_chin
- removed joint camera_joint_face
- removed joint camera_joint_left
- removed joint camera_joint_rearDown
- removed joint camera_joint_right
- removed joint camera_laserscan_joint_left
- removed joint camera_laserscan_joint_right
- removed joint camera_optical_joint_chin
- removed joint camera_optical_joint_face
- removed joint camera_optical_joint_left
- removed joint camera_optical_joint_rearDown
- removed joint camera_optical_joint_right
- removed joint ultraSound_joint_face
- removed joint ultraSound_joint_left
- removed joint ultraSound_joint_right

Commit message: modify the mesh loading using os

File: files/go1_description/go1.urdf (robot description, URDF)
Before this commit: robot go1, 31 links, 30 joints
Links:
- link FL_calf: geometry collision box size=0.213 0.016 0.016; visual mesh filename=package://go1_description/meshes/calf.dae scale=1 1 1
- link FL_hip: geometry collision cylinder length=0.04 radius=0.046; visual mesh filename=package://go1_description/meshes/hip.dae scale=1 1 1
- link FL_thigh: geometry collision box size=0.213 0.0245 0.034; visual mesh filename=package://go1_description/meshes/thigh.dae scale=1 1 1
- link FR_calf: geometry collision box size=0.213 0.016 0.016; visual mesh filename=package://go1_description/meshes/calf.dae scale=1 1 1
- link FR_hip: geometry collision cylinder length=0.04 radius=0.046; visual mesh filename=package://go1_description/meshes/hip.dae scale=1 1 1
- link FR_thigh: geometry collision box size=0.213 0.0245 0.034; visual mesh filename=package://go1_description/meshes/thigh_mirror.dae scale=1 1 1
- link RL_calf: geometry collision box size=0.213 0.016 0.016; visual mesh filename=package://go1_description/meshes/calf.dae scale=1 1 1
- link RL_hip: geometry collision cylinder length=0.04 radius=0.046; visual mesh filename=package://go1_description/meshes/hip.dae scale=1 1 1
- link RL_thigh: geometry collision box size=0.213 0.0245 0.034; visual mesh filename=package://go1_description/meshes/thigh.dae scale=1 1 1
- link RR_calf: geometry collision box size=0.213 0.016 0.016; visual mesh filename=package://go1_description/meshes/calf.dae scale=1 1 1
- link RR_hip: geometry collision cylinder length=0.04 radius=0.046; visual mesh filename=package://go1_description/meshes/hip.dae scale=1 1 1
- link RR_thigh: geometry collision box size=0.213 0.0245 0.034; visual mesh filename=package://go1_description/meshes/thigh_mirror.dae scale=1 1 1
- link trunk: geometry collision box size=0.3762 0.0935 0.114; visual mesh filename=package://go1_description/meshes/trunk.dae scale=1 1 1

File: files/solo_description/solo12.urdf (robot description, URDF)
Before this commit: robot solo, 17 links, 16 joints
Links:
- link FL_LOWER_LEG: geometry collision mesh filename=package://solo_description/mesh/without_foot/solo_lower_leg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; visual mesh filename=package://solo_description/mesh/without_foot/solo_lower_leg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
- link FL_SHOULDER: geometry collision mesh filename=package://solo_description/mesh/solo12/solo12_hip_fe_fl.stl; visual mesh filename=package://solo_description/mesh/solo12/solo12_hip_fe_fl.stl
- link FL_UPPER_LEG: geometry collision mesh filename=package://solo_description/mesh/without_foot/solo_upper_leg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; visual mesh filename=package://solo_description/mesh/without_foot/solo_upper_leg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
- link FR_LOWER_LEG: geometry collision mesh filename=package://solo_description/mesh/without_foot/solo_lower_leg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; visual mesh filename=package://solo_description/mesh/without_foot/solo_lower_leg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
- link FR_SHOULDER: geometry collision mesh filename=package://solo_description/mesh/solo12/solo12_hip_fe_fr.stl; visual mesh filename=package://solo_description/mesh/solo12/solo12_hip_fe_fr.stl
- link FR_UPPER_LEG: geometry collision mesh filename=package://solo_description/mesh/without_foot/solo_upper_leg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; visual mesh filename=package://solo_description/mesh/without_foot/solo_upper_leg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
- link HL_LOWER_LEG: geometry collision mesh filename=package://solo_description/mesh/without_foot/solo_lower_leg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; visual mesh filename=package://solo_description/mesh/without_foot/solo_lower_leg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
- link HL_SHOULDER: geometry collision mesh filename=package://solo_description/mesh/solo12/solo12_hip_fe_hl.stl; visual mesh filename=package://solo_description/mesh/solo12/solo12_hip_fe_hl.stl
- link HL_UPPER_LEG: geometry collision mesh filename=package://solo_description/mesh/without_foot/solo_upper_leg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; visual mesh filename=package://solo_description/mesh/without_foot/solo_upper_leg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
- link HR_LOWER_LEG: geometry collision mesh filename=package://solo_description/mesh/without_foot/solo_lower_leg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; visual mesh filename=package://solo_description/mesh/without_foot/solo_lower_leg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
- link HR_SHOULDER: geometry collision mesh filename=package://solo_description/mesh/solo12/solo12_hip_fe_hr.stl; visual mesh filename=package://solo_description/mesh/solo12/solo12_hip_fe_hr.stl
- link HR_UPPER_LEG: geometry collision mesh filename=package://solo_description/mesh/without_foot/solo_upper_leg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; visual mesh filename=package://solo_description/mesh/without_foot/solo_upper_leg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
- link base_link: geometry collision mesh filename=package://solo_description/mesh/solo12/solo_12_base.stl; visual mesh filename=package://solo_description/mesh/solo12/solo_12_base.stl

File: files/spot_description/spot.urdf (robot description, URDF)
Before this commit: robot spot, 20 links, 19 joints
Links:
- link base_link: geometry visual mesh filename=package://spot_description/meshes/base/visual/body.obj
- link body: geometry collision mesh filename=package://spot_description/meshes/base/collision/body_colli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; visual mesh filename=package://spot_description/meshes/base/visual/body.obj
- link front_left_hip: geometry visual mesh filename=package://spot_description/meshes/base/visual/front_left_hi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
- link front_left_lower_leg: geometry collision mesh filename=package://spot_description/meshes/base/collision/left_lower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; collision sphere radius=0.036
- link front_left_upper_leg: geometry collision mesh filename=package://spot_description/meshes/base/collision/left_upper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; visual mesh filename=package://spot_description/meshes/base/visual/front_left_up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
- link front_right_hip: geometry visual mesh filename=package://spot_description/meshes/base/visual/front_right_h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
- link front_right_lower_leg: geometry collision mesh filename=package://spot_description/meshes/base/collision/right_lowe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; collision sphere radius=0.036
- link front_right_upper_leg: geometry collision mesh filename=package://spot_description/meshes/base/collision/right_uppe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; visual mesh filename=package://spot_description/meshes/base/visual/front_right_u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
- link rear_left_hip: geometry visual mesh filename=package://spot_description/meshes/base/visual/rear_left_hip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
- link rear_left_lower_leg: geometry collision mesh filename=package://spot_description/meshes/base/collision/left_lower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; collision sphere radius=0.036
- link rear_left_upper_leg: geometry collision mesh filename=package://spot_description/meshes/base/collision/left_upper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; visual mesh filename=package://spot_description/meshes/base/visual/rear_left_upp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
- link rear_right_hip: geometry visual mesh filename=package://spot_description/meshes/base/visual/rear_right_hi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
- link rear_right_lower_leg: geometry collision mesh filename=package://spot_description/meshes/base/collision/right_lowe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; collision sphere radius=0.036
- link rear_right_upper_leg: geometry collision mesh filename=package://spot_description/meshes/base/collision/right_uppe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; visual mesh filename=package://spot_description/meshes/base/visual/rear_right_up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
