Commit message: modify the urdf and config files

File: files/spot_description/spot.urdf (robot description, URDF)
Before this commit: robot spot, 20 links, 19 joints
Links:
- link base_link: geometry visual mesh filename=/home/khorshidi/git/system_identification/files/spot_descri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

Commit message: modify spot files

File: files/spot_description/spot.urdf (robot description, URDF)
Before this commit: robot spot, 20 links, 19 joints
Links:
- link base_link: mass 32.86 -> 16.52

Commit message: final version for the submitted paper

File: files/spot_description/spot.urdf (robot description, URDF)
Before this commit: robot spot, 20 links, 19 joints
Links:
- removed link fl_foot
- removed link fr_foot
- removed link rl_foot
- removed link rr_foot
- added link front_left_foot, mass 0.0
- added link front_right_foot, mass 0.0
- added link rear_left_foot, mass 0.0
- added link rear_right_foot, mass 0.0
Joints:
- removed joint fl_ankle
- removed joint fr_ankle
- removed joint rl_ankle
- removed joint rr_ankle
- added joint front_left_ankle: type fixed, parent front_left_lower_leg, child front_left_foot, origin xyz=0 0 -0.35 rpy=0 0 0, limit lower=-10 upper=10 effort=1000 velocity=1000
- added joint front_right_ankle: type fixed, parent front_right_lower_leg, child front_right_foot, origin xyz=0 0 -0.35 rpy=0 0 0, limit lower=-10 upper=10 effort=1000 velocity=1000
- added joint rear_left_ankle: type fixed, parent rear_left_lower_leg, child rear_left_foot, origin xyz=0 0 -0.35 rpy=0 0 0, limit lower=-10 upper=10 effort=1000 velocity=1000
- added joint rear_right_ankle: type fixed, parent rear_right_lower_leg, child rear_right_foot, origin xyz=0 0 -0.35 rpy=0 0 0, limit lower=-10 upper=10 effort=1000 velocity=1000
